File: Audio_sch.kicad_sch (KiCad schematic)
At the start: 35 parts, among them J1 Audio_InL, J2 Audio_InR, J3 Audio_OutL, J4 Audio_OutR, U1 OPA2132, U2 CS3310, U3 Daisy Seed, U4 CS3310, U5 NE5532

Commit message: New Routing
Parts:
- added C33, C34: 100n, Capacitor_SMD:C_0805_2012Metric_Pad1.18x1.45mm_HandSolder, symbol Device:C
- added J10: Jack In Right, symbol Connector:Barrel_Jack_Switch
- added J11: Conn_01x02_Socket, symbol Connector:Conn_01x02_Socket
- added J12: ~, symbol Connector:Conn_01x02_Socket
- added J9: Jack In Left, symbol Connector:Barrel_Jack_Switch
Connections:
- net GNDA: now also C33.2, C34.2
- net at R10.1, U3.18 (OUTL): now also C34.1
- net at R9.1, U3.19 (OUTR): now also C33.1
- new net: J10.3, J11.1 (Pin_1), J9.2
- new net: J11.2 (Pin_2), J9.1, J9.3
- new net: J10.1, J12.1 (Pin_1)
- new net: J10.2, J12.2 (Pin_2)
Other:
- moved on the sheet: C1, C2, C3, C4, C5, C6, J1, J2, R1, R10, R11, R18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
