File: PENDAII-Hardware.kicad_pcb (KiCad board)
At the start: 2 copper layers, 84 x 89 mm, 89 parts, among them J1 Audio_InL, J2 Audio_InR, J3 Audio_OutL, J4 Audio_OutR, J5 Switch 1, J6 Switch 2, J7 Jack MIDI, J8 Alim 12V, SW1 Encoder0, SW2 Encoder1, SW3 Encoder2, SW4 Encoder3, U1 OPA2132, U10 L79L05_SOT89, U11 AMS1117-3.3, U2 CS3310, U3 Daisy Seed, U4 CS3310, U5 NE5532, U6 TFT 2p, U7 H11L1, U8 L78L05_SOT89, U9 L78L05_SOT89

Commit message: New Routing
Parts:
- added C33: 100n, Capacitor_SMD:C_0805_2012Metric_Pad1.18x1.45mm_HandSolder, B.Cu at (49.9, 73.4)
- added C34: 100n, Capacitor_SMD:C_0805_2012Metric_Pad1.18x1.45mm_HandSolder, B.Cu at (52.6, 73.5)
- R20, R21, R22, R23, R24: value 22k -> 47k
Routing:
- net GNDA: track 98.8 -> 109.0 mm
- net Net-(U3A-OUTL): track 91.1 -> 94.3 mm
- net Net-(U3A-OUTR): track 90.3 -> 93.4 mm
- net PB8/D11: track 60.5 -> 62.2 mm
- net PB9/D12: track 53.4 -> 54.5 mm
- net PG10/D7: track 69.6 -> 70.4 mm
Other:
- board text added: "PENDA II V 1.0.2"
- board text removed: "PENDA II V 1.0.1"
