File: UI_sch.kicad_sch (KiCad schematic)
At the start: 21 parts, among them J5 Switch 1, J6 Switch 2, J7 Jack MIDI, SW1 Encoder0, SW2 Encoder1, SW3 Encoder2, SW4 Encoder3, U2 CS3310, U3 Daisy Seed, U4 CS3310, U6 TFT 2p, U7 H11L1

Commit message: New Routing
Parts:
- R20, R21, R22, R23, R24: value 22k -> 47k
Changed lines of the file:
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@@
 			)
 		)
-		(property "Value" "22k"
+		(property "Value" "47k"
 			(at 156.21 77.4699 0)
 			(effects
@@
 			)
 		)
-		(property "Value" "22k"
+		(property "Value" "47k"
 			(at 165.1 77.4699 0)
 			(effects
@@
 			)
 		)
-		(property "Value" "22k"
+		(property "Value" "47k"
 			(at 137.16 77.4699 0)
 			(effects
@@
 			)
 		)
-		(property "Value" "22k"
+		(property "Value" "47k"
 			(at 173.99 77.4699 0)
 			(effects
@@
 			)
 		)
-		(property "Value" "22k"
+		(property "Value" "47k"
 			(at 146.05 77.4699 0)
 			(effects
